File: schematics/PSLab.kicad_pcb (KiCad board)
At the start: 4 copper layers, 99 x 53.3 mm, 182 parts, among them J1 DoublePins, J11 Li-Ion Battery, J2 Power Pins, J3 Wave Generator, J4 I2C, J5 I2C, J6 ESP01, J7 UART, J9 SPI, P1 SDCard, Q1 MMBT3906, Q2 MMBT3904, Q3 MMBT3906, Q4 Q_NMOS_DGS, SW1 BOOT, SW2 MCLR Reset, SW3 USB_C - Generic, U1 LDFM33PUR, U10 TL082, U11 TL082, U12 MCP4728, U13 MCP6S21, U14 MCP6S21, U15 CP2102N, U16 SP0503BAHT, U18 LTC4040, U19 TC1240A, U2 74HC126, U3 PIC24EP256GP204, U4 DS1307Z+, U5 TC7660, U7 LM324, U8 TL082, U9 TL082, X2 32.768 kHz, Y1 12 MHz

Commit message: chore: pull request actions
Parts:
- J1: moved to F.Cu
- moved J2 17.1 mm to (157.0, 62.8), turned to 90 degrees
- moved J9 12.8 mm to (113.8, 62.8), turned to 90 degrees
- moved J7 3.08 mm to (136.7, 111.1)
- moved J1 2.87 mm to (187.5, 67.9), turned to 0 degrees
- moved J11 1.29 mm to (94.8, 110.2)
- moved TP4 1.21 mm to (188.2, 64.9)
- moved FID3 1.17 mm to (188.0, 62.4)
- moved FID1 1.14 mm to (94.0, 107.2)
- moved BT1 1.13 mm to (175.6, 106.0)
- moved BT2 1.12 mm to (175.5, 106.3)
- moved FID2 1.00 mm to (188.0, 106.0)
- moved J3 0.79 mm to (149.4, 111.0)
- moved SW3 0.63 mm to (92.8, 75.5)
- moved P1 0.47 mm to (99.3, 92.4)
- moved J5 0.43 mm to (144.3, 62.8)
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Connections:
- J1 pad 1: /VOL -> AVSS
- J1 pad 10: AVSS -> MIC
- J1 pad 11: CH3.GAIN -> AVSS
- J1 pad 12: AVSS -> CH3.GAIN
- J1 pad 13: CH3 -> AVSS
- J1 pad 14: AVSS -> CH3
- J1 pad 15: CH2 -> AVSS
- J1 pad 16: AVSS -> CH2
- J1 pad 17: CH1 -> AVSS
- J1 pad 18: AVSS -> CH1
- J1 pad 19: ACH1 -> AVSS
- J1 pad 2: AVSS -> /VOL
- J1 pad 20: AVSS -> ACH1
- J1 pad 21: LA4 -> AVSS
- J1 pad 22: AVSS -> LA4
- J1 pad 23: LA3 -> AVSS
- J1 pad 24: AVSS -> LA3
- J1 pad 25: LA2 -> AVSS
- J1 pad 26: AVSS -> LA2
- J1 pad 27: LA1 -> AVSS
- J1 pad 28: AVSS -> LA1
- J1 pad 3: /RES -> AVSS
- J1 pad 4: AVSS -> /RES
- J1 pad 5: /CAP -> AVSS
- J1 pad 6: AVSS -> /CAP
- J1 pad 7: FQy -> AVSS
- J1 pad 8: AVSS -> FQy
- J1 pad 9: MIC -> AVSS
- J2 pad 1: PVS1 -> AVSS
- J2 pad 2: AVSS -> PCS
- J2 pad 3: PVS2 -> AVSS
- J2 pad 4: AVSS -> PVS3
- J2 pad 5: PVS3 -> AVSS
- J2 pad 6: AVSS -> PVS2
- J2 pad 7: PCS -> AVSS
- J2 pad 8: AVSS -> PVS1
- J9 pad 1: +3V3 -> SPI.CS
- J9 pad 2: AVSS -> SDI
- J9 pad 3: SCK -> SDO
- J9 pad 4: SDO -> SCK
- J9 pad 5: SDI -> AVSS
- J9 pad 6: SPI.CS -> +3V3
Routing:
- net VR+: track 83.2 -> 0.00 mm, vias 4 -> 0
- net +6V: track 0.00 -> 83.2 mm, vias 0 -> 4
- net VR-: track 62.3 -> 2.30 mm, vias 3 -> 0
- net -6V: track 0.00 -> 60.0 mm, vias 0 -> 3
- net TxD2: track 0.00 -> 23.9 mm, vias 0 -> 1
- net RxD2: track 23.9 -> 0.00 mm, vias 1 -> 0
- net SPI.CS: track 34.8 -> 15.7 mm
- net FQy: track 45.5 -> 27.8 mm
- net SDI: track 59.4 -> 43.2 mm
- net ACH1: track 25.0 -> 12.0 mm
- net AVSS: track 316.8 -> 304.5 mm
- net CH2: track 32.5 -> 20.3 mm
- net CH1: track 28.6 -> 17.6 mm
- net PVS2: track 16.3 -> 6.89 mm
- net VDDA: track 0.02 -> 6.73 mm
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