File: schematics/PSLab.sch (KiCad schematic (older format))
At the start: 183 parts, among them J1 DoublePins, J11 Li-Ion Battery, J2 Power Pins, J3 Wave Generator, J4 I2C, J5 I2C, J6 ESP01, J7 UART, J9 SPI, P1 SDCard, Q1 MMBT3906, Q2 MMBT3904, Q3 MMBT3906, Q4 Q_NMOS_DGS, SW1 BOOT, SW2 MCLR Reset, SW3 USB_C - Generic, U1 LDFM33PUR, U10 TL082, U11 TL082, U12 MCP4728, U13 MCP6S21, U14 MCP6S21, U15 CP2102N, U16 SP0503BAHT, U18 LTC4040, U19 TC1240A, U2 74HC126, U3 PIC24EP256GP204, U4 DS1307Z+, U5 TC7660, U7 LM324, U8 TL082, U9 TL082, X2 32.768 kHz, Y1 12 MHz

Commit message: test
Other:
- note added: "PR Test"
Changed lines of the file:
@@
 Data
 89 50 4E 47 0D 0A 1A 0A 00 00 00 0D 49 48 44 52 00 00 02 08 00 00 00 CC 08 03 00 00 00 21 C4 AB
-DA 00 00 00 03 73 42 49 54 08 08 08 DB E1 4F E0 00 00 03 00 50 4C 54 45 02 00 00 FF FF E2 79 5D
+DA 00 00 00 03 73 42 49 54 08 08 08 DB E1 4F E0 00 00 03 00 50 4C 54 45 01 00 00 FF FF E2 79 5D
 9D 28 5D A5 28 7D CE E2 FF FF 81 5D B6 A5 EA FF C6 99 A5 28 99 E2 FF EA D6 59 5D C2 C6 FF FF 59
 B6 F2 FF FF F2 A5 7D A5 28 5D C6 E2 B6 B6 81 CE FF FF CE C6 81 7D D6 55 5D A1 59 7D BE F6 F6 F6
@@
 F6 99 D2 CE 40 9D D6 EA EE F6 40 5D A5 28 5D BA 7D D2 DE 55 AE DE 28 75 C2 CA DA EA 99 AA B6 65
 C2 DE 85 A5 CA 4C 4C 4C A1 A1 A1 3C 3C 3C 61 65 69 A5 B2 BE 85 A1 CE 91 99 A1 EE F2 F2 7D 81 81
-B6 BE C6 91 91 91 7D 7D 81 50 79 B6 C2 C2 C2 99 B2 7D 5D B6 DE FA FA FA 4A AB 90 C2 00 00 00 01
+B6 BE C6 91 91 91 7D 7D 81 50 79 B6 C2 C2 C2 99 B2 7D 5D B6 DE FA FA FA 76 CF DF 8C 00 00 00 01
 74 52 4E 53 00 40 E6 D8 66 00 00 15 08 49 44 41 54 78 9C ED 9D 7B 80 15 D5 79 C0 67 99 A5 31 A6
 26 05 83 EC 2E FB 76 60 9B 44 F6 01 BB CA 43 77 F7 C6 18 1F 10 31 36 1B 5D 4C 82 69 D6 24 D6 A0
@@
 	0    -1   -1   0
 $EndComp
+Text Notes 13175 5875 0    197  ~ 0
+PR Test
 $EndSCHEMATC
